Commit message: configurable beam length

File: kuka_kl_support/urdf/kl100_2_macro.xacro (robot description, xacro)
@@ -1,20 +1,55 @@
 <?xml version="1.0" encoding="UTF-8"?>
 <robot xmlns:xacro="http://www.ros.org/wiki/xacro">
-  <xacro:macro name="kl100_2_links" params="prefix">
-    <!-- links -->
+  <!-- Recursive macro: place beam sections along the beam -->
+  <xacro:macro name="kl100_2_beam_sections" params="count x spacing">
+    <xacro:if value="${count > 0}">
+      <visual>
+        <origin xyz="${x} 0.0075 0.042" rpy="0 0 0"/>
+        <geometry>
+          <mesh filename="package://kuka_kl_support/meshes/kl100_2/visual/beam_section.dae"/>
+        </geometry>
+      </visual>
+      <xacro:kl100_2_beam_sections count="${count - 1}" x="${x + spacing}" spacing="${spacing}"/>
+    </xacro:if>
+  </xacro:macro>
+  <xacro:macro name="kl100_2_links" params="prefix rated_travel:=2.0">
+    <!-- Beam geometry constants derived from the repeatable CAD section -->
+    <xacro:property name="segment_length" value="0.25"/>
+    <xacro:property name="beam_end_length" value="0.3475"/>
+    <xacro:property name="num_beam_sections" value="${int(rated_travel / segment_length)}"/>
+    <xacro:property name="beam_section_start" value="${-(num_beam_sections - 1) * segment_length / 2}"/>
+    <xacro:property name="beam_left_edge" value="${beam_section_start - segment_length / 2}"/>
+    <xacro:property name="beam_right_edge" value="${beam_section_start + (num_beam_sections - 0.5) * segment_length}"/>
+    <xacro:property name="beam_length" value="${num_beam_sections * segment_length + 2 * beam_end_length}"/>
+    <!-- Inertia scaling (reference: 2.695m beam, 500kg) -->
+    <xacro:property name="ref_beam_length" value="2.695"/>
+    <xacro:property name="lr" value="${beam_length / ref_beam_length}"/>
     <link name="${prefix}base_link">
       <inertial>
-        <origin rpy="0.0 0.0 0.0" xyz="0.0 0.0 0.0"/>
-        <mass value="500.0"/>
-        <inertia ixx="8" ixy="0.0" ixz="0.0" iyy="190" iyz="0.0" izz="190"/>
+        <origin rpy="0 0 0" xyz="0 0 0"/>
+        <mass value="${500.0 * lr}"/>
+        <inertia ixx="${8 * lr}" ixy="0" ixz="0" iyy="${190 * lr * lr * lr}" iyz="0" izz="${190 * lr * lr * lr}"/>
       </inertial>
+      <!-- Repeatable beam sections from the CAD export -->
+      <xacro:kl100_2_beam_sections count="${num_beam_sections}" x="${beam_section_start}" spacing="${segment_length}"/>
+      <!-- Right beam end piece -->
       <visual>
+        <origin xyz="${beam_right_edge} -0.001 0.357" rpy="0 0 ${pi}"/>
         <geometry>
-          <mesh filename="package://kuka_kl_support/meshes/kl100_2/visual/base_link.dae"/>
+          <mesh filename="package://kuka_kl_support/meshes/kl100_2/visual/beam_end_right.dae"/>
         </geometry>
       </visual>
+      <!-- Left beam end piece -->
+      <visual>
+        <origin xyz="${beam_left_edge} -0.001 0.357" rpy="0 0 ${pi}"/>
+        <geometry>
+          <mesh filename="package://kuka_kl_support/meshes/kl100_2/visual/beam_end_left.dae"/>
+        </geometry>
+      </visual>
+      <!-- Collision - parametric box covering the whole beam envelope -->
       <collision>
+        <origin xyz="0 0.1675 0.1035" rpy="0 0 0"/>
         <geometry>
-          <mesh filename="package://kuka_kl_support/meshes/kl100_2/collision/base_link.stl"/>
+          <box size="${beam_length} 0.697 0.207"/>
         </geometry>
       </collision>
@@ -22,7 +57,7 @@
     <link name="${prefix}link_1">
       <inertial>
-        <origin rpy="0.0 0.0 0.0" xyz="0.0 0.0 0.0"/>
+        <origin rpy="0 0 0" xyz="0 0 0"/>
         <mass value="43.0"/>
-        <inertia ixx="1.03" ixy="0.0" ixz="0.0" iyy="1.135" iyz="0.0" izz="1.517"/>
+        <inertia ixx="1.03" ixy="0" ixz="0" iyy="1.135" iyz="0" izz="1.517"/>
       </inertial>
       <visual>
@@ -38,17 +73,16 @@
     </link>
   </xacro:macro>
-  <xacro:macro name="kl100_2_joints" params="prefix robot_base_link *origin">
-    <!-- joints -->
+  <xacro:macro name="kl100_2_joints" params="prefix robot_base_link rated_travel:=2.0 *origin">
     <joint name="${prefix}joint_1" type="prismatic">
       <parent link="${prefix}base_link"/>
       <child link="${prefix}link_1"/>
-      <origin rpy="0.0 0.0 0.0" xyz="0.0 0.0 0.0"/>
+      <origin rpy="0 0 0" xyz="0 0 0"/>
       <axis xyz="1 0 0"/>
-      <limit lower="-1.0" upper="1.0" effort="702.0" velocity="2.5"/>
+      <limit lower="${-rated_travel / 2}" upper="${rated_travel / 2}" effort="702.0" velocity="2.5"/>
     </joint>
     <joint name="${prefix}link_1-${robot_base_link}" type="fixed">
       <parent link="${prefix}link_1"/>
       <child link="${robot_base_link}"/>
-      <origin rpy="0.0 0.0 0.0" xyz="0.0 0.0 0.356"/>
+      <origin rpy="0 0 0" xyz="0 0 0.356"/>
     </joint>
   </xacro:macro>

File: kuka_resources/urdf/robot_with_external_axis_template.urdf.xacro (robot description, xacro)
@@ -31,4 +31,5 @@
   <xacro:arg name="kl_model" default="kl100_2"/>
   <xacro:arg name="kl_ros2_control_joints_macro" default="kuka_kl_ros2_control_joints"/>
+  <xacro:arg name="kl_rated_travel" default="2.0"/>
   <xacro:arg name="rsi_xml_config_file" default=""/>
   <xacro:arg name="gazebo_controller_config_path" default="config/fake_hardware_config_6_axis_kl.yaml"/>
@@ -48,4 +49,5 @@
   <xacro:property name="kl_model_joints_macro_name" value="${kl_model_value + '_joints'}"/>
   <xacro:property name="kl_ros2_control_joints_macro_name" value="$(arg kl_ros2_control_joints_macro)"/>
+  <xacro:property name="kl_rated_travel_value" value="$(arg kl_rated_travel)"/>
   <xacro:property name="kl_full_prefix" value="${prefix_value + kl_prefix_value}"/>
   <!-- Include urdf macro files -->
@@ -69,9 +71,9 @@
   </joint>
   <!-- external axis links -->
-  <xacro:call macro="${kl_model_links_macro_name}" prefix="${kl_full_prefix}"/>
+  <xacro:call macro="${kl_model_links_macro_name}" prefix="${kl_full_prefix}" rated_travel="${kl_rated_travel_value}"/>
   <!-- robot links -->
   <xacro:call macro="${robot_model_macro_name}" prefix="$(arg prefix)" package_name="$(arg robot_support_package)"/>
   <!-- external axis joints -->
-  <xacro:call macro="${kl_model_joints_macro_name}" prefix="${kl_full_prefix}" robot_base_link="$(arg prefix)base_link">
+  <xacro:call macro="${kl_model_joints_macro_name}" prefix="${kl_full_prefix}" robot_base_link="$(arg prefix)base_link" rated_travel="${kl_rated_travel_value}">
     <origin xyz="$(arg x) $(arg y) $(arg z)" rpy="$(arg roll) $(arg pitch) $(arg yaw)"/>
   </xacro:call>

Commit message: use scaling for beam section (no recursive xacro); add missing meshes+energy supply system; param for energy system placement

File: kuka_kl_support/urdf/kl100_2_macro.xacro (robot description, xacro)
@@ -1,17 +1,5 @@
 <?xml version="1.0" encoding="UTF-8"?>
 <robot xmlns:xacro="http://www.ros.org/wiki/xacro">
-  <!-- Recursive macro: place beam sections along the beam -->
-  <xacro:macro name="kl100_2_beam_sections" params="count x spacing">
-    <xacro:if value="${count > 0}">
-      <visual>
-        <origin xyz="${x} 0.0075 0.042" rpy="0 0 0"/>
-        <geometry>
-          <mesh filename="package://kuka_kl_support/meshes/kl100_2/visual/beam_section.dae"/>
-        </geometry>
-      </visual>
-      <xacro:kl100_2_beam_sections count="${count - 1}" x="${x + spacing}" spacing="${spacing}"/>
-    </xacro:if>
-  </xacro:macro>
-  <xacro:macro name="kl100_2_links" params="prefix rated_travel:=2.0">
+  <xacro:macro name="kl100_2_links" params="prefix rated_travel:=2.0 energy_supply_placement:=side">
     <!-- Beam geometry constants derived from the repeatable CAD section -->
     <xacro:property name="segment_length" value="0.25"/>
@@ -22,5 +10,13 @@
     <xacro:property name="beam_right_edge" value="${beam_section_start + (num_beam_sections - 0.5) * segment_length}"/>
     <xacro:property name="beam_length" value="${num_beam_sections * segment_length + 2 * beam_end_length}"/>
-    <!-- Inertia scaling (reference: 2.695m beam, 500kg) -->
+    <xacro:property name="beam_end_outer_extension" value="0.3075"/>
+    <xacro:property name="beam_section_scale_x" value="${num_beam_sections}"/>
+    <xacro:property name="installation_area_length" value="${beam_length}"/>
+    <xacro:property name="installation_area_start" value="${(beam_left_edge + beam_right_edge - installation_area_length) / 2.0}"/>
+    <!-- Side energy supply length mapping from rated travel (m) -->
+    <xacro:property name="energy_supply_mesh_length" value="0.305"/>
+    <xacro:property name="energy_supply_length" value="${0.467 + 0.25 * int(rated_travel / 0.5)}"/>
+    <xacro:property name="energy_supply_scale_x" value="${energy_supply_length / energy_supply_mesh_length}"/>
+    <!-- Inertia scaling (reference 2.695m beam, 500kg) -->
     <xacro:property name="ref_beam_length" value="2.695"/>
     <xacro:property name="lr" value="${beam_length / ref_beam_length}"/>
@@ -31,6 +27,27 @@
         <inertia ixx="${8 * lr}" ixy="0" ixz="0" iyy="${190 * lr * lr * lr}" iyz="0" izz="${190 * lr * lr * lr}"/>
       </inertial>
-      <!-- Repeatable beam sections from the CAD export -->
-      <xacro:kl100_2_beam_sections count="${num_beam_sections}" x="${beam_section_start}" spacing="${segment_length}"/>
+      <!-- Mesh1 from original base_link.dae - installation area preserving COLLADA material -->
+      <visual>
+        <origin xyz="${installation_area_start} -0.181 0.0" rpy="0 0 0"/>
+        <geometry>
+          <mesh filename="package://kuka_kl_support/meshes/kl100_2/visual/installation_area.dae" scale="${installation_area_length / 2.695} 1 1"/>
+        </geometry>
+      </visual>
+      <!-- Beam sections from the CAD export as a single scaled mesh -->
+      <visual>
+        <origin xyz="0 0.0075 0.042" rpy="0 0 0"/>
+        <geometry>
+          <mesh filename="package://kuka_kl_support/meshes/kl100_2/visual/beam_section.dae" scale="${beam_section_scale_x} 1 1"/>
+        </geometry>
+      </visual>
+      <!-- Mesh6/Mesh7 reworked use a single side energy-supply visual if placement is side -->
+      <xacro:if value="${energy_supply_placement == 'side'}">
+        <visual>
+          <origin xyz="${beam_left_edge - beam_end_outer_extension} -0.001 0.356" rpy="0 0 ${pi}"/>
+          <geometry>
+            <mesh filename="package://kuka_kl_support/meshes/kl100_2/visual/energy_supply_section.dae" scale="${energy_supply_scale_x} 1 1"/>
+          </geometry>
+        </visual>
+      </xacro:if>
       <!-- Right beam end piece -->
       <visual>
@@ -47,4 +64,13 @@
         </geometry>
       </visual>
+      <!-- Mesh5 from original base_link.dae - energy supply station shown only for side placement -->
+      <xacro:if value="${energy_supply_placement == 'side'}">
+        <visual>
+          <origin xyz="0.212 0.485 0.0305" rpy="0 0 ${pi}"/>
+          <geometry>
+            <mesh filename="package://kuka_kl_support/meshes/kl100_2/visual/energy_supply_station.dae"/>
+          </geometry>
+        </visual>
+      </xacro:if>
       <!-- Collision - parametric box covering the whole beam envelope -->
       <collision>

Commit message: add collision meshes for the specific base link subparts

File: kuka_kl_support/urdf/kl100_2_macro.xacro (robot description, xacro)
@@ -73,11 +73,43 @@
         </visual>
       </xacro:if>
-      <!-- Collision - parametric box covering the whole beam envelope -->
+      <!-- Collision meshes mirror the visual composition with coarse STL assets -->
       <collision>
-        <origin xyz="0 0.1675 0.1035" rpy="0 0 0"/>
+        <origin xyz="${installation_area_start} -0.181 0.0" rpy="0 0 0"/>
         <geometry>
-          <box size="${beam_length} 0.697 0.207"/>
+          <mesh filename="package://kuka_kl_support/meshes/kl100_2/collision/installation_area.stl" scale="${installation_area_length / 2.695} 1 1"/>
         </geometry>
       </collision>
+      <collision>
+        <origin xyz="0 0.0075 0.042" rpy="0 0 0"/>
+        <geometry>
+          <mesh filename="package://kuka_kl_support/meshes/kl100_2/collision/beam_section.stl" scale="${beam_section_scale_x} 1 1"/>
+        </geometry>
+      </collision>
+      <collision>
+        <origin xyz="${beam_right_edge} -0.001 0.357" rpy="0 0 ${pi}"/>
+        <geometry>
+          <mesh filename="package://kuka_kl_support/meshes/kl100_2/collision/beam_end_right.stl"/>
+        </geometry>
+      </collision>
+      <collision>
+        <origin xyz="${beam_left_edge} -0.001 0.357" rpy="0 0 ${pi}"/>
+        <geometry>
+          <mesh filename="package://kuka_kl_support/meshes/kl100_2/collision/beam_end_left.stl"/>
+        </geometry>
+      </collision>
+      <xacro:if value="${energy_supply_placement == 'side'}">
+        <collision>
+          <origin xyz="${beam_left_edge - beam_end_outer_extension} -0.001 0.356" rpy="0 0 ${pi}"/>
+          <geometry>
+            <mesh filename="package://kuka_kl_support/meshes/kl100_2/collision/energy_supply_section.stl" scale="${energy_supply_scale_x} 1 1"/>
+          </geometry>
+        </collision>
+        <collision>
+          <origin xyz="0.212 0.485 0.0305" rpy="0 0 ${pi}"/>
+          <geometry>
+            <mesh filename="package://kuka_kl_support/meshes/kl100_2/collision/energy_supply_station.stl"/>
+          </geometry>
+        </collision>
+      </xacro:if>
     </link>
     <link name="${prefix}link_1">

Commit message: config file for family/model-specific params; add new params

File: kuka_kl_support/urdf/kl100_2_macro.xacro (robot description, xacro)
@@ -1,5 +1,10 @@
 <?xml version="1.0" encoding="UTF-8"?>
 <robot xmlns:xacro="http://www.ros.org/wiki/xacro">
-  <xacro:macro name="kl100_2_links" params="prefix rated_travel:=2.0 energy_supply_placement:=side">
+  <xacro:macro name="kl100_2_links" params="prefix rated_travel:=2.0 kl_config_file">
+    <xacro:property name="kl_config" value="${xacro.load_yaml(kl_config_file)}"/>
+    <xacro:property name="energy_supply_placement" value="${kl_config['energy_supply_placement']}"/>
+    <xacro:property name="installation_area" value="${kl_config['installation_area']}"/>
+    <xacro:property name="carriage_rotation" value="${kl_config['carriage_rotation']}"/>
+    <xacro:property name="energy_supply_left" value="${kl_config['energy_supply_left']}"/>
     <!-- Beam geometry constants derived from the repeatable CAD section -->
     <xacro:property name="segment_length" value="0.25"/>
@@ -28,10 +33,12 @@
       </inertial>
       <!-- Mesh1 from original base_link.dae - installation area preserving COLLADA material -->
-      <visual>
-        <origin xyz="${installation_area_start} -0.181 0.0" rpy="0 0 0"/>
-        <geometry>
-          <mesh filename="package://kuka_kl_support/meshes/kl100_2/visual/installation_area.dae" scale="${installation_area_length / 2.695} 1 1"/>
-        </geometry>
-      </visual>
+      <xacro:if value="${installation_area}">
+         <visual>
+            <origin xyz="${installation_area_start} -0.181 0.0" rpy="0 0 0"/>
+            <geometry>
+               <mesh filename="package://kuka_kl_support/meshes/kl100_2/visual/installation_area.dae" scale="${installation_area_length / 2.695} 1 1"/>
+            </geometry>
+         </visual>
+      </xacro:if>
       <!-- Beam sections from the CAD export as a single scaled mesh -->
       <visual>
@@ -131,16 +138,16 @@
     </link>
   </xacro:macro>
-  <xacro:macro name="kl100_2_joints" params="prefix robot_base_link rated_travel:=2.0 *origin">
+  <xacro:macro name="kl100_2_joints" params="prefix robot_base_link rated_travel:=2.0 pedestal_size:=0.0 offset:=0.0 robot_position:=0.0 *origin">
     <joint name="${prefix}joint_1" type="prismatic">
       <parent link="${prefix}base_link"/>
       <child link="${prefix}link_1"/>
-      <origin rpy="0 0 0" xyz="0 0 0"/>
+      <origin rpy="0 0 0" xyz="${offset} 0 0"/>
       <axis xyz="1 0 0"/>
-      <limit lower="${-rated_travel / 2}" upper="${rated_travel / 2}" effort="702.0" velocity="2.5"/>
+      <limit lower="${-rated_travel / 2 + offset}" upper="${rated_travel / 2 + offset}" effort="702.0" velocity="2.5"/>
     </joint>
     <joint name="${prefix}link_1-${robot_base_link}" type="fixed">
       <parent link="${prefix}link_1"/>
       <child link="${robot_base_link}"/>
-      <origin rpy="0 0 0" xyz="0 0 0.356"/>
+      <origin rpy="0 0 ${-1.57079633 + robot_position}" xyz="0 0 ${0.356 + pedestal_size}"/>
     </joint>
   </xacro:macro>

File: kuka_resources/urdf/robot_with_external_axis_template.urdf.xacro (robot description, xacro)
@@ -32,5 +32,8 @@
   <xacro:arg name="kl_ros2_control_joints_macro" default="kuka_kl_ros2_control_joints"/>
   <xacro:arg name="kl_rated_travel" default="2.0"/>
-  <xacro:arg name="kl_energy_supply_placement" default="side"/>
+  <xacro:arg name="kl_pedestal_size" default="0.0"/>
+  <xacro:arg name="kl_offset" default="0.0"/>
+  <xacro:arg name="kl_robot_position" default="0.0"/>
+  <xacro:arg name="kl_config_file" default=""/>
   <xacro:arg name="rsi_xml_config_file" default=""/>
   <xacro:arg name="gazebo_controller_config_path" default="config/fake_hardware_config_6_axis_kl.yaml"/>
@@ -51,4 +54,7 @@
   <xacro:property name="kl_ros2_control_joints_macro_name" value="$(arg kl_ros2_control_joints_macro)"/>
   <xacro:property name="kl_rated_travel_value" value="$(arg kl_rated_travel)"/>
+  <xacro:property name="kl_pedestal_size_value" value="$(arg kl_pedestal_size)"/>
+  <xacro:property name="kl_offset_value" value="$(arg kl_offset)"/>
+  <xacro:property name="kl_robot_position_value" value="$(arg kl_robot_position)"/>
   <xacro:property name="kl_full_prefix" value="${prefix_value + kl_prefix_value}"/>
   <!-- Include urdf macro files -->
@@ -72,9 +78,9 @@
   </joint>
   <!-- external axis links -->
-  <xacro:call macro="${kl_model_links_macro_name}" prefix="${kl_full_prefix}" rated_travel="${kl_rated_travel_value}" energy_supply_placement="$(arg kl_energy_supply_placement)"/>
+  <xacro:call macro="${kl_model_links_macro_name}" prefix="${kl_full_prefix}" rated_travel="${kl_rated_travel_value}" kl_config_file="$(arg kl_config_file)"/>
   <!-- robot links -->
   <xacro:call macro="${robot_model_macro_name}" prefix="$(arg prefix)" package_name="$(arg robot_support_package)"/>
   <!-- external axis joints -->
-  <xacro:call macro="${kl_model_joints_macro_name}" prefix="${kl_full_prefix}" robot_base_link="$(arg prefix)base_link" rated_travel="${kl_rated_travel_value}">
+  <xacro:call macro="${kl_model_joints_macro_name}" prefix="${kl_full_prefix}" robot_base_link="$(arg prefix)base_link" rated_travel="${kl_rated_travel_value}" pedestal_size="${kl_pedestal_size_value}" offset="${kl_offset_value}" robot_position="${kl_robot_position_value}">
     <origin xyz="$(arg x) $(arg y) $(arg z)" rpy="$(arg roll) $(arg pitch) $(arg yaw)"/>
   </xacro:call>
